Commit message: Add IMU link and Gazebo IMU plugin to bumperbot URDF

File: bumperbot_description/urdf/bumperbot.urdf.xacro (robot description, xacro)
@@ -139,4 +139,34 @@
         <origin rpy="0 0 0" xyz ="-0.04755 0 -0.0275"/>
     </joint>
+    <link name="imu_link">
+      <inertial>
+        <origin xyz="-0.00552433659106688 0.000168210391520346 0.000514000497342681" rpy="0 0 0" />
+        <mass value="0.000528415362211671" />
+        <inertia ixx="1.46176048428261E-08" ixy="1.40015117949421E-10" ixz="-1.99633872937403E-12"
+                 iyy="8.59662482954888E-09" iyz="7.52375112767959E-12"
+                 izz="2.30279421279312E-08" />
+      </inertial>
+      <visual>
+        <origin xyz="0 0 0" rpy="0 0 0"/>
+        <geometry>
+          <mesh filename="package://bumperbot_description/meshes/imu_link.STL"/>
+        </geometry>
+        <material name="">
+          <color rgba="0.792156862745098 0.819607843137255 0.933333333333333 1" />
+        </material>
+      </visual>
+      <collision>
+        <origin xyz="0 0 0" rpy="0 0 0"/>
+        <geometry>
+          <mesh filename="package://bumperbot_description/meshes/imu_link.STL"/>
+        </geometry>
+      </collision>
+    </link>
+    <joint name="imu_joint" type="fixed">
+        <origin xyz="0 0 0.0698986241758014" rpy="0 0 0" />
+        <parent link="base_link" />
+        <child link="imu_link" />
+        <axis xyz="0 0 0" />
+    </joint>
     <!--link name="can_link">
          <visual>

File: bumperbot_description/urdf/bumperbot_gazebo.xacro (robot description, xacro)
@@ -34,15 +34,73 @@
        <maxVel>0.1</maxVel>
    </gazebo>
+   <!--ROS2 control plugin-->
    <gazebo>
+    <!--ROS2 Humble-->
      <xacro:if value="$(arg is_ignition)">
        <plugin filename="ign_ros2_control-system" name="ign_ros2_control::IgnitionROS2ControlPlugin">
           <parameters>$(find bumperbot_controller)/config/bumperbot_controller.yaml</parameters>
        </plugin>
+       <plugin filename="ignition-gazebo-imu-system" name="ignition::gazebo::systems::Imu">
+       </plugin>
      </xacro:if>
+     <!--ROS2 Iron or above-->
      <xacro:unless value="$(arg is_ignition)">
         <plugin filename="gz_ros2_control-system" name="gz_ros2_control::GazeboSimROS2ControlPlugin">
            <parameters>$(find bumperbot_controller)/config/bumperbot_controller.yaml</parameters>
         </plugin>
+        <plugin filename="gz-sim-imu-system" name="gz::sim::system::Imu">
+       </plugin>
      </xacro:unless>
    </gazebo>
+   <!-- IMU -->
+  <gazebo reference="imu_link">
+    <sensor name="imu" type="imu">
+        <always_on>true</always_on>
+        <update_rate>100</update_rate>
+        <gz_frame_id>imu_link</gz_frame_id>
+        <topic>imu</topic>
+        <imu>
+          <angular_velocity>
+            <x>
+              <noise type="gaussian">
+                <mean>0.0</mean>
+                <stddev>2e-4</stddev>
+              </noise>
+            </x>
+            <y>
+              <noise type="gaussian">
+                <mean>0.0</mean>
+                <stddev>2e-4</stddev>
+              </noise>
+            </y>
+            <z>
+              <noise type="gaussian">
+                <mean>0.0</mean>
+                <stddev>2e-4</stddev>
+              </noise>
+            </z>
+          </angular_velocity>
+          <linear_acceleration>
+            <x>
+              <noise type="gaussian">
+                <mean>0.0</mean>
+                <stddev>1.7e-2</stddev>
+              </noise>
+            </x>
+            <y>
+              <noise type="gaussian">
+                <mean>0.0</mean>
+                <stddev>1.7e-2</stddev>
+              </noise>
+            </y>
+            <z>
+              <noise type="gaussian">
+                <mean>0.0</mean>
+                <stddev>1.7e-2</stddev>
+              </noise>
+            </z>
+          </linear_acceleration>
+        </imu>
+    </sensor>
+  </gazebo>
 </robot>

Commit message: Update robot description: add laser mesh and integrate into URDF and gazebo configs

File: bumperbot_description/urdf/bumperbot.urdf.xacro (robot description, xacro)
@@ -2,4 +2,6 @@
 <robot name="bumperbot" xmlns:xacro="http://www.ros.org/wiki/xacro">
    <xacro:arg name="is_ignition" default="true"/>
+   <!-- Load Simulated or Real Hardware Interfaces -->
+   <xacro:arg name="is_sim" default="true"/>
     <!-- Include Gazebo Parameters -->
     <xacro:include filename="$(find bumperbot_description)/urdf/bumperbot_gazebo.xacro" />
@@ -20,4 +22,5 @@
                 <mesh filename="package://bumperbot_description/meshes/base_link.STL"/>
             </geometry>
+            <material name="black"/>
         </visual>
         <collision>
@@ -31,5 +34,5 @@
         <parent link="base_footprint"/>
         <child link="base_link"/>
-        <origin rpy="0 0 0" xyz="0 0 0.033"/>
+        <origin xyz="0 0 0.033" rpy="0 0 0"/>
     </joint>
     <link name="wheel_right_link">
@@ -42,21 +45,22 @@
         </inertial>
         <visual>
-            <origin rpy="1.57 0 0" xyz = "0 0 0"/>
+            <origin xyz = "0 0 0" rpy="1.57 0 0" />
             <geometry>
                  <mesh filename="package://bumperbot_description/meshes/wheel_right_link.STL"/>
             </geometry>
-        </visual>
-        <collision>
-           <origin xyz="0 -015 0" rpy="1.57 0 0"/>
-           <geometry>
-             <sphere radius="0.033"/>
+            <material name="blue"/>
+        </visual>
+        <collision>
+           <origin xyz="0 -0.015 0" rpy="1.57 0 0" />
+           <geometry>
+             <sphere radius="0.033" />
            </geometry>
         </collision>
     </link>
     <joint name="wheel_right_joint" type="continuous">
-        <parent link="base_link"/>
-        <child link="wheel_right_link"/>
+        <origin xyz="0 -0.0701101849418637 0" rpy="0 0 0" />
+        <parent link="base_link" />
+        <child link="wheel_right_link" />
         <axis xyz="0 1 0"/>
-        <origin rpy="0 0 0" xyz="0 -0.07 0"/>
     </joint>
     <link name="wheel_left_link">
@@ -69,11 +73,12 @@
         </inertial>
         <visual>
-            <origin rpy="-1.57 0 0" xyz = "0 0 0"/>
+            <origin xyz="0 0 0" rpy="-1.57 0 0" />
             <geometry>
                  <mesh filename="package://bumperbot_description/meshes/wheel_left_link.STL"/>
             </geometry>
-        </visual>
-        <collision>
-           <origin xyz="0 015 0" rpy="1.57 0 0"/>
+            <material name="blue"/>
+        </visual>
+        <collision>
+           <origin xyz="0 0.015 0" rpy="-1.57 0 0" />
            <geometry>
              <sphere radius="0.033"/>
@@ -82,8 +87,8 @@
     </link>
     <joint name="wheel_left_joint" type="continuous">
+        <origin xyz="0 0.0701101849418642 0" rpy="0 0 0" />
         <parent link="base_link"/>
         <child link="wheel_left_link"/>
         <axis xyz="0 1 0"/>
-        <origin rpy="0 0 0" xyz="0 0.07 0"/>
     </joint>
     <link name="caster_front_link">
@@ -100,4 +105,5 @@
                   <mesh filename="package://bumperbot_description/meshes/caster_front_link.STL"/>
              </geometry>
+             <material name="silver"/>
         </visual>
         <collision>
@@ -126,4 +132,5 @@
                   <mesh filename="package://bumperbot_description/meshes/caster_rear_link.STL"/>
              </geometry>
+             <material name="silver"/>
         </visual>
         <collision>
@@ -152,7 +159,5 @@
           <mesh filename="package://bumperbot_description/meshes/imu_link.STL"/>
         </geometry>
-        <material name="">
-          <color rgba="0.792156862745098 0.819607843137255 0.933333333333333 1" />
-        </material>
+        <material name="blue"/>
       </visual>
       <collision>
@@ -169,4 +174,42 @@
         <axis xyz="0 0 0" />
     </joint>
+    <link name="laser_link">
+      <inertial>
+        <origin xyz="-0.011945780406062 -0.000381929217680526 -0.0170649378129477" rpy="0 0 0" />
+        <mass value="0.073084435549317" />
+        <inertia ixx="1.96074931730795E-05" ixy="-3.62091076640009E-07" ixz="4.28230084046735E-07" iyy="2.40983835136327E-05" iyz="1.50180909250652E-08" izz="4.14184164228595E-05" />
+      </inertial>
+      <visual>
+        <origin xyz="0 0 0" rpy="0 0 0"/>
+        <geometry>
+          <mesh filename="package://bumperbot_description/meshes/laser_link.STL"/>
+        </geometry>
+        <material name="dark_grey"/>
+      </visual>
+      <collision>
+        <origin xyz="0 0 0" rpy="0 0 0"/>
+        <geometry>
+          <mesh filename="package://bumperbot_description/meshes/laser_link.STL"/>
+        </geometry>
+      </collision>
+    </link>
+    <joint name="laser_joint" type="fixed">
+        <origin xyz="0.0 0.0 0.1208" rpy="0 0 3.14" />
+        <parent link="base_link" />
+        <child link="laser_link" />
+        <axis xyz="0 0 0" />
+    </joint>
+    <material name="blue">
+      <color rgba="0 0 1 1"/>
+    </material>
+    <material name="black">
+      <color rgba="0 0 0 1"/>
+    </material>
+    <material name="silver">
+      <color rgba="0.79 0.82 0.93 1"/>
+    </material>
+    <material name="dark_grey">
+      <color rgba="0.3 0.3 0.3 1"/>
+    </material>
     <!--link name="can_link">
          <visual>

File: bumperbot_description/urdf/bumperbot_gazebo.xacro (robot description, xacro)
@@ -1,2 +1,3 @@
+<?xml version="1.0"?>
 <robot name ="bumperbot" xmlns:xacro="http://www.ros.org/wiki/xacro">
    <gazebo reference="wheel_right_link">
@@ -43,4 +44,7 @@
        <plugin filename="ignition-gazebo-imu-system" name="ignition::gazebo::systems::Imu">
        </plugin>
+       <plugin filename="ignition-gazebo-sensors-system" name="ignition::gazebo::systems::Sensors">
+         <render_engine>ogre2</render_engine>
+       </plugin>
      </xacro:if>
      <!--ROS2 Iron or above-->
@@ -50,4 +54,7 @@
         </plugin>
         <plugin filename="gz-sim-imu-system" name="gz::sim::system::Imu">
+       </plugin>
+       <plugin filename="gz-sim-sensors-system" name="gz::sim::systems::Sensors">
+         <render_engine>ogre2</render_engine>
        </plugin>
      </xacro:unless>
@@ -104,3 +111,32 @@
     </sensor>
   </gazebo>
+  <gazebo reference="laser_link">
+    <sensor name="lidar" type="gpu_ray">
+      <always_on>true</always_on>
+      <visualize>true</visualize>
+      <topic>scan</topic>
+      <update_rate>5</update_rate>
+      <gz_frame_id>laser_link</gz_frame_id>
+      <ray>
+        <scan>
+           <horizontal>
+             <samples>360</samples>
+             <resolution>1.0</resolution>
+             <min_angle>0.0</min_angle>
+             <max_angle>6.28</max_angle>
+           </horizontal>
+        </scan>
+        <range>
+         <min>0.12</min>
+         <max>12.0</max>
+         <resolution>0.02</resolution>
+      </range>
+      <noise>
+        <type>gaussian</type>
+        <mean>0.0</mean>
+        <stddev>0.01</stddev>
+      </noise>
+      </ray>
+    </sensor>
+  </gazebo>
 </robot>
